Commit message: Created models for links

File: ros2/src/wx200_control/urdf/test.urdf (robot description, URDF)
Before this commit: robot wx200, 7 links, 6 joints
Links:
- link elbow: geometry visual box size=0.200 0.025 0.025; visual cylinder length=0.1 radius=0.025
- link shoulder: geometry visual box size=0.050 0.025 0.025; visual box size=0.200 0.025 0.025
- link waist: geometry visual cylinder length=0.06325 radius=0.05
- link wrist_angle: geometry visual cylinder length=0.1 radius=0.025
- link wrist_roll: geometry visual box size=0.025 0.025 0.06605; visual cylinder length=0.065 radius=0.025
